Commit message: remove all instance of '_arm'

File: xacro/doublepanda_default.urdf.xacro (robot description, xacro)
@@ -1,16 +1,16 @@
 <?xml version="1.0" encoding="utf-8"?>
-<robot xmlns:xacro="http://www.ros.org/wiki/xacro" name="panda">
+<robot xmlns:xacro="http://www.ros.org/wiki/xacro" name="doublepanda_default">
   <xacro:arg name="gazebo" default="true"/>
   <xacro:include filename="@CMAKE_BINARY_DIR@/xacro/main.xacro">
     <xacro:arg name="gazebo" value="${gazebo}"/>
   </xacro:include>
-  <xacro:include filename="@CMAKE_BINARY_DIR@/xacro/pandaA_arm.xacro">
+  <xacro:include filename="@CMAKE_BINARY_DIR@/xacro/pandaA.xacro">
     <xacro:arg name="gazebo" value="${gazebo}"/>
   </xacro:include>
-  <xacro:include filename="@CMAKE_BINARY_DIR@/xacro/pandaB_arm.xacro">
+  <xacro:include filename="@CMAKE_BINARY_DIR@/xacro/pandaB.xacro">
     <xacro:arg name="gazebo" value="${gazebo}"/>
   </xacro:include>
   <xacro:main connected_to='world'/>
-  <xacro:panda_armA xyz="0 +1 0" connected_to='main_link'/>
-  <xacro:panda_armB xyz="0 -1 0" connected_to='main_link'/>
+  <xacro:pandaA xyz="0 +1 0" connected_to='main_link'/>
+  <xacro:pandaB xyz="0 -1 0" connected_to='main_link'/>
 </robot>

File: xacro/foot.xacro (robot description, xacro)
@@ -1,4 +1,4 @@
 <?xml version="1.0" encoding="utf-8"?>
-<robot xmlns:xacro="http://www.ros.org/wiki/xacro" name="hand">
+<robot xmlns:xacro="http://www.ros.org/wiki/xacro" name="panda_foot_part">
   <xacro:macro name="foot" params="connected_to:='' ns:='' rpy:='0 0 0' xyz:='0 0 0' ">
     <xacro:unless value="${connected_to == ''}">

File: xacro/main.xacro (robot description, xacro)
@@ -1,4 +1,4 @@
 <?xml version='1.0' encoding='utf-8'?>
-<robot xmlns:xacro="http://www.ros.org/wiki/xacro" name="panda">
+<robot xmlns:xacro="http://www.ros.org/wiki/xacro" name="panda_main_part">
   <xacro:macro name="main" params="arm_id:='main' package_name:='franka_gazebo' connected_to:='' xyz:='0 0 0' rpy:='0 0 0'">
     <xacro:unless value="${not connected_to}">

File: xacro/pandaA.xacro (robot description, xacro)
@@ -1,5 +1,5 @@
 <?xml version='1.0' encoding='utf-8'?>
-<robot xmlns:xacro="http://www.ros.org/wiki/xacro" name="panda">
-  <xacro:macro name="panda_armA" params="arm_id:='panda' package_name:='franka_gazebo' connected_to:='' xyz:='0 0 0' rpy:='0 0 0'">
+<robot xmlns:xacro="http://www.ros.org/wiki/xacro" name="panda_manipulatorA_part">
+  <xacro:macro name="pandaA" params="arm_id:='panda' package_name:='franka_gazebo' connected_to:='' xyz:='0 0 0' rpy:='0 0 0'">
     <xacro:unless value="${not connected_to}">
       <!-- <link name="${connected_to}"/>-->
@@ -13,5 +13,5 @@
     <xacro:if value="$(arg gazebo)">
       <!-- Gazebo Tags -->
-      <xacro:include filename="pandaA_arm.gazebo.xacro"/>
+      <xacro:include filename="pandaA.gazebo.xacro"/>
     </xacro:if>
     <link name="${arm_id}_linkA0">

File: xacro/pandaB.xacro (robot description, xacro)
@@ -1,5 +1,5 @@
 <?xml version='1.0' encoding='utf-8'?>
-<robot xmlns:xacro="http://www.ros.org/wiki/xacro" name="panda">
-  <xacro:macro name="panda_armB" params="arm_id:='panda' package_name:='franka_gazebo' connected_to:='' xyz:='0 0 0' rpy:='0 0 0'">
+<robot xmlns:xacro="http://www.ros.org/wiki/xacro" name="panda_manipulatorB_part">
+  <xacro:macro name="pandaB" params="arm_id:='panda' package_name:='franka_gazebo' connected_to:='' xyz:='0 0 0' rpy:='0 0 0'">
     <xacro:unless value="${not connected_to}">
       <!-- <link name="${connected_to}"/>-->
@@ -13,5 +13,5 @@
     <xacro:if value="$(arg gazebo)">
       <!-- Gazebo Tags -->
-      <xacro:include filename="pandaB_arm.gazebo.xacro"/>
+      <xacro:include filename="pandaB.gazebo.xacro"/>
     </xacro:if>
     <link name="${arm_id}_linkB0">

File: xacro/panda_default.urdf.xacro (robot description, xacro)
@@ -1,12 +1,12 @@
 <?xml version="1.0" encoding="utf-8"?>
-<robot xmlns:xacro="http://www.ros.org/wiki/xacro" name="panda">
+<robot xmlns:xacro="http://www.ros.org/wiki/xacro" name="panda_default">
   <xacro:arg name="gazebo" default="true"/>
   <xacro:include filename="@CMAKE_BINARY_DIR@/xacro/main.xacro">
     <xacro:arg name="gazebo" value="${gazebo}"/>
   </xacro:include>
-  <xacro:include filename="@CMAKE_BINARY_DIR@/xacro/pandaA_arm.xacro">
+  <xacro:include filename="@CMAKE_BINARY_DIR@/xacro/pandaA.xacro">
     <xacro:arg name="gazebo" value="${gazebo}"/>
   </xacro:include>
   <xacro:main connected_to='world'/>
-  <xacro:panda_armA xyz="0 0 0" connected_to='main_link'/>
+  <xacro:pandaA xyz="0 0 0" connected_to='main_link'/>
 </robot>

File: xacro/panda_foot.urdf.xacro (robot description, xacro)
@@ -1,14 +1,14 @@
 <?xml version="1.0" encoding="utf-8"?>
-<robot xmlns:xacro="http://www.ros.org/wiki/xacro" name="panda">
+<robot xmlns:xacro="http://www.ros.org/wiki/xacro" name="panda_foot">
   <xacro:arg name="gazebo" default="true"/>
   <xacro:include filename="@CMAKE_BINARY_DIR@/xacro/main.xacro">
     <xacro:arg name="gazebo" value="${gazebo}"/>
   </xacro:include>
-  <xacro:include filename="@CMAKE_BINARY_DIR@/xacro/pandaA_arm.xacro">
+  <xacro:include filename="@CMAKE_BINARY_DIR@/xacro/pandaA.xacro">
     <xacro:arg name="gazebo" value="${gazebo}"/>
   </xacro:include>
   <xacro:include filename="@CMAKE_BINARY_DIR@/xacro/foot.xacro"/>
   <xacro:main connected_to='world'/>
-  <xacro:panda_armA xyz="0 0 0" connected_to='main_link'/>
+  <xacro:pandaA xyz="0 0 0" connected_to='main_link'/>
   <xacro:foot ns="panda" rpy="0 0 ${-pi/4}" connected_to="panda_linkA8"/>
 </robot>

File: xacro/panda_hand.urdf.xacro (robot description, xacro)
@@ -1,14 +1,14 @@
 <?xml version="1.0" encoding="utf-8"?>
-<robot xmlns:xacro="http://www.ros.org/wiki/xacro" name="panda">
+<robot xmlns:xacro="http://www.ros.org/wiki/xacro" name="panda_hand">
   <xacro:arg name="gazebo" default="true"/>
   <xacro:include filename="@CMAKE_BINARY_DIR@/xacro/main.xacro">
     <xacro:arg name="gazebo" value="${gazebo}"/>
   </xacro:include>
-  <xacro:include filename="@CMAKE_BINARY_DIR@/xacro/pandaA_arm.xacro">
+  <xacro:include filename="@CMAKE_BINARY_DIR@/xacro/pandaA.xacro">
     <xacro:arg name="gazebo" value="${gazebo}"/>
   </xacro:include>
   <xacro:include filename="$(find franka_gazebo)/robots/hand.xacro"/>
   <xacro:main connected_to='world'/>
-  <xacro:panda_armA xyz="0 0 0" connected_to='main_link'/>
+  <xacro:pandaA xyz="0 0 0" connected_to='main_link'/>
   <xacro:hand ns="panda" rpy="0 0 ${-pi/4}" connected_to="panda_linkA8"/>
 </robot>

Commit message: use simple collision shapes

File: xacro/doublepanda_default.urdf.xacro (robot description, xacro)
@@ -12,5 +12,5 @@
   </xacro:include>
   <xacro:main connected_to='world'/>
-  <xacro:pandaA xyz="0 +1 0" connected_to='main_link'/>
+  <xacro:pandaA xyz="0 +1 0" connected_to='main_link' safety_distance="0.03"/>
   <xacro:pandaB xyz="0 -1 0" connected_to='main_link'/>
 </robot>

File: xacro/pandaA_old.xacro (robot description, xacro)
@@ -1,6 +1,4 @@
 <?xml version='1.0' encoding='utf-8'?>
 <robot xmlns:xacro="http://www.ros.org/wiki/xacro" name="panda_manipulatorA_part">
-  <!-- safety_distance: Minimum safety distance in [m] by which the collision volumes are expanded and which is enforced during robot motions -->
-  <!-- arm_id: Namespace of the panda arm. Serves to differentiate between arms in case of multiple instances. -->
   <xacro:macro name="pandaA" params="arm_id:='panda' package_name:='franka_gazebo' connected_to:='' xyz:='0 0 0' rpy:='0 0 0' safety_distance:=0">
     <xacro:unless value="${not connected_to}">
@@ -33,19 +31,7 @@
       </visual>
       <collision>
-        <origin xyz="-0.075 0 0.06" rpy="0 ${pi/2} 0"/>
-        <geometry>
-          <cylinder radius="${0.06+safety_distance}" length="0.03" />
-        </geometry>
-      </collision>
-      <collision>
-        <origin xyz="-0.06 0 0.06" rpy="0 0 0"/>
-        <geometry>
-          <sphere radius="${0.06+safety_distance}" />
-        </geometry>
-      </collision>
-      <collision>
-        <origin xyz="-0.09 0 0.06" rpy="0 0 0"/>
-        <geometry>
-          <sphere radius="${0.06+safety_distance}" />
+        <origin xyz="0 0 0" rpy="0 0 0"/>
+        <geometry>
+          <mesh filename="package://${package_name}/meshes/collision/link0.stl"/>
         </geometry>
       </collision>
@@ -67,19 +53,7 @@
       </visual>
       <collision>
-        <origin xyz="0 0 -0.1915" rpy="0 0 0"/>
-        <geometry>
-          <cylinder radius="${0.06+safety_distance}" length="0.2830" />
-        </geometry>
-      </collision>
-      <collision>
-        <origin xyz="0 0 -0.333" rpy="0 0 0"/>
-        <geometry>
-          <sphere radius="${0.06+safety_distance}" />
-        </geometry>
-      </collision>
-      <collision>
-        <origin xyz="0 0 -0.05" rpy="0 0 0"/>
-        <geometry>
-          <sphere radius="${0.06+safety_distance}" />
+        <origin xyz="0 0 0" rpy="0 0 0"/>
+        <geometry>
+          <mesh filename="package://${package_name}/meshes/collision/link1.stl"/>
         </geometry>
       </collision>
@@ -111,17 +85,5 @@
         <origin xyz="0 0 0" rpy="0 0 0"/>
         <geometry>
-          <cylinder radius="${0.06+safety_distance}" length="0.12" />
-        </geometry>
-      </collision>
-      <collision>
-        <origin xyz="0 0 -0.06" rpy="0 0 0"/>
-        <geometry>
-          <sphere radius="${0.06+safety_distance}" />
-        </geometry>
-      </collision>
-      <collision>
-        <origin xyz="0 0 0.06" rpy="0 0 0"/>
-        <geometry>
-          <sphere radius="${0.06+safety_distance}" />
+          <mesh filename="package://${package_name}/meshes/collision/link2.stl"/>
         </geometry>
       </collision>
@@ -151,19 +113,7 @@
       </visual>
       <collision>
-        <origin xyz="0 0 -0.145" rpy="0 0 0"/>
-        <geometry>
-          <cylinder radius="${0.06+safety_distance}" length="0.15" />
-        </geometry>
-      </collision>
-      <collision>
-        <origin xyz="0 0 -0.22" rpy="0 0 0"/>
-        <geometry>
-          <sphere radius="${0.06+safety_distance}" />
-        </geometry>
-      </collision>
-      <collision>
-        <origin xyz="0 0 -0.07" rpy="0 0 0"/>
-        <geometry>
-          <sphere radius="${0.06+safety_distance}" />
+        <origin xyz="0 0 0" rpy="0 0 0"/>
+        <geometry>
+          <mesh filename="package://${package_name}/meshes/collision/link3.stl"/>
         </geometry>
       </collision>
@@ -195,17 +145,5 @@
         <origin xyz="0 0 0" rpy="0 0 0"/>
         <geometry>
-          <cylinder radius="${0.06+safety_distance}" length="0.12" />
-        </geometry>
-      </collision>
-      <collision>
-        <origin xyz="0 0 0.06" rpy="0 0 0"/>
-        <geometry>
-          <sphere radius="${0.06+safety_distance}" />
-        </geometry>
-      </collision>
-      <collision>
-        <origin xyz="0 0 -0.06" rpy="0 0 0"/>
-        <geometry>
-          <sphere radius="${0.06+safety_distance}" />
+          <mesh filename="package://${package_name}/meshes/collision/link4.stl"/>
         </geometry>
       </collision>
@@ -235,37 +173,7 @@
       </visual>
       <collision>
-        <origin xyz="0 0 -0.26" rpy="0 0 0"/>
-        <geometry>
-          <cylinder radius="${0.06+safety_distance}" length="0.1" />
-        </geometry>
-      </collision>
-      <collision>
-        <origin xyz="0 0 -0.31" rpy="0 0 0"/>
-        <geometry>
-          <sphere radius="${0.06+safety_distance}" />
-        </geometry>
-      </collision>
-      <collision>
-        <origin xyz="0 0 -0.21" rpy="0 0 0"/>
-        <geometry>
-          <sphere radius="${0.06+safety_distance}" />
-        </geometry>
-      </collision>
-      <collision>
-        <origin xyz="0 0.08 -0.13" rpy="0 0 0"/>
-        <geometry>
-          <cylinder radius="${0.025+safety_distance}" length="0.14" />
-        </geometry>
-      </collision>
-      <collision>
-        <origin xyz="0 0.08 -0.06" rpy="0 0 0"/>
-        <geometry>
-          <sphere radius="${0.025+safety_distance}" />
-        </geometry>
-      </collision>
-      <collision>
-        <origin xyz="0 0.08 -0.20" rpy="0 0 0"/>
-        <geometry>
-          <sphere radius="${0.025+safety_distance}" />
+        <origin xyz="0 0 0" rpy="0 0 0"/>
+        <geometry>
+          <mesh filename="package://${package_name}/meshes/collision/link5.stl"/>
         </geometry>
       </collision>
@@ -295,19 +203,7 @@
       </visual>
       <collision>
-        <origin xyz="0 0 -0.03" rpy="0 0 0"/>
-        <geometry>
-          <cylinder radius="${0.05+safety_distance}" length="0.08" />
-        </geometry>
-      </collision>
-      <collision>
-        <origin xyz="0 0 0.01" rpy="0 0 0"/>
-        <geometry>
-          <sphere radius="${0.05+safety_distance}" />
-        </geometry>
-      </collision>
-      <collision>
-        <origin xyz="0 0 -0.07" rpy="0 0 0"/>
-        <geometry>
-          <sphere radius="${0.05+safety_distance}" />
+        <origin xyz="0 0 0" rpy="0 0 0"/>
+        <geometry>
+          <mesh filename="package://${package_name}/meshes/collision/link6.stl"/>
         </geometry>
       </collision>
@@ -337,19 +233,7 @@
       </visual>
       <collision>
-        <origin xyz="0 0 0.01" rpy="0 0 0"/>
-        <geometry>
-          <cylinder radius="${0.04+safety_distance}" length="0.14" />
-        </geometry>
-      </collision>
-      <collision>
-        <origin xyz="0 0 0.08" rpy="0 0 0"/>
-        <geometry>
-          <sphere radius="${0.04+safety_distance}"  />
-        </geometry>
-      </collision>
-      <collision>
-        <origin xyz="0 0 -0.06" rpy="0 0 0"/>
-        <geometry>
-          <sphere radius="${0.04+safety_distance}"  />
+        <origin xyz="0 0 0" rpy="0 0 0"/>
+        <geometry>
+          <mesh filename="package://${package_name}/meshes/collision/link7.stl"/>
         </geometry>
       </collision>
@@ -363,24 +247,5 @@
       <limit effort="12" lower="-2.8973" upper="2.8973" velocity="2.6100"/>
     </joint>
-    <link name="${arm_id}_linkA8">
-      <collision>
-        <origin xyz="0.0424 0.0424 -0.0250" rpy="${pi} ${pi/2} ${pi/2}"/>
-        <geometry>
-          <cylinder radius="${0.03+safety_distance}"  length="0.01" />
-        </geometry>
-      </collision>
-      <collision>
-        <origin xyz="0.0424 0.0424 -0.02" rpy="0 0 0"/>
-        <geometry>
-          <sphere radius="${0.03+safety_distance}"  />
-        </geometry>
-      </collision>
-      <collision>
-        <origin xyz="0.0424 0.0424 -0.03" rpy="0 0 0"/>
-        <geometry>
-          <sphere radius="${0.03+safety_distance}"  />
-        </geometry>
-      </collision>
-    </link>
+    <link name="${arm_id}_linkA8"/>
     <joint name="${arm_id}_jointA8" type="fixed">
       <origin rpy="0 0 0" xyz="0 0 0.107"/>

File: xacro/panda_default.urdf.xacro (robot description, xacro)
@@ -9,4 +9,4 @@
   </xacro:include>
   <xacro:main connected_to='world'/>
-  <xacro:pandaA xyz="0 0 0" connected_to='main_link'/>
+  <xacro:pandaA xyz="0 0 0" connected_to='main_link' safety_distance="0.03"/>
 </robot>

File: xacro/panda_foot.urdf.xacro (robot description, xacro)
@@ -10,5 +10,5 @@
   <xacro:include filename="@CMAKE_BINARY_DIR@/xacro/foot.xacro"/>
   <xacro:main connected_to='world'/>
-  <xacro:pandaA xyz="0 0 0" connected_to='main_link'/>
+  <xacro:pandaA xyz="0 0 0" connected_to='main_link' safety_distance="0.03"/>
   <xacro:foot ns="panda" rpy="0 0 ${-pi/4}" connected_to="panda_linkA8"/>
 </robot>

File: xacro/panda_hand.urdf.xacro (robot description, xacro)
@@ -10,5 +10,5 @@
   <xacro:include filename="$(find franka_gazebo)/robots/hand.xacro"/>
   <xacro:main connected_to='world'/>
-  <xacro:pandaA xyz="0 0 0" connected_to='main_link'/>
+  <xacro:pandaA xyz="0 0 0" connected_to='main_link' safety_distance="0.03"/>
   <xacro:hand ns="panda" rpy="0 0 ${-pi/4}" connected_to="panda_linkA8"/>
 </robot>
